File: mfos_vco/first_page.kicad_sch (KiCad schematic)
At the start: 49 parts, among them Q1 PN4391, Q1Ar1 2N3904, Q1Br1 2N3904, U1 OP275, U2 TL072, U3 SSM2210

Commit message: FINISHED ROUTING
Parts:
- Q1: footprint Package_TO_SOT_THT:TO-92L_Inline -> Package_TO_SOT_THT:TO-92L_Inline_Wide
- Q1Ar1, Q1Br1: footprint Package_TO_SOT_THT:TO-92_Inline -> Package_TO_SOT_THT:TO-92L_Inline_Wide
Connections:
- net R2P2: no longer R2.3, R65.1
- new net R2P3: R2.3, R65.1
Changed lines of the file:
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@@
 	)
 	(junction
+		(at 40.64 71.12)
+		(diameter 0)
+		(color 0 0 0 0)
+	)
+	(junction
 		(at 273.05 97.79)
 		(diameter 0)
@@
 	)
 	(junction
+		(at 43.18 58.42)
+		(diameter 0)
+		(color 0 0 0 0)
+	)
+	(junction
+		(at 81.28 58.42)
+		(diameter 0)
+		(color 0 0 0 0)
+	)
+	(junction
+		(at 81.28 71.12)
+		(diameter 0)
+		(color 0 0 0 0)
+	)
+	(junction
 		(at 106.68 119.38)
 		(diameter 0)
@@
 	(wire
 		(pts
+			(xy 81.28 71.12) (xy 90.17 71.12)
+		)
+		(stroke
+			(width 0)
+			(type default)
+		)
+	)
+	(wire
+		(pts
 			(xy 120.65 100.33) (xy 120.65 107.95)
 		)
@@
 	(wire
 		(pts
+			(xy 40.64 71.12) (xy 52.07 71.12)
+		)
+		(stroke
+			(width 0)
+			(type default)
+		)
+	)
+	(wire
+		(pts
 			(xy 78.74 124.46) (xy 83.82 124.46)
 		)
@@
 	(wire
 		(pts
+			(xy 81.28 58.42) (xy 90.17 58.42)
+		)
+		(stroke
+			(width 0)
+			(type default)
+		)
+	)
+	(wire
+		(pts
 			(xy 157.48 101.6) (xy 157.48 143.51)
 		)
@@
 	(wire
 		(pts
+			(xy 81.28 57.15) (xy 81.28 58.42)
+		)
+		(stroke
+			(width 0)
+			(type default)
+		)
+	)
+	(wire
+		(pts
 			(xy 100.33 119.38) (xy 106.68 119.38)
 		)
@@
 	(wire
 		(pts
+			(xy 81.28 68.58) (xy 81.28 71.12)
+		)
+		(stroke
+			(width 0)
+			(type default)
+		)
+	)
+	(wire
+		(pts
 			(xy 143.51 101.6) (xy 143.51 110.49)
 		)
@@
 	(wire
 		(pts
-			(xy 72.39 58.42) (xy 90.17 58.42)
+			(xy 72.39 58.42) (xy 81.28 58.42)
 		)
 		(stroke
@@
 	(wire
 		(pts
+			(xy 40.64 68.58) (xy 40.64 71.12)
+		)
+		(stroke
+			(width 0)
+			(type default)
+		)
+	)
+	(wire
+		(pts
 			(xy 83.82 109.22) (xy 83.82 116.84)
 		)
@@
 	(wire
 		(pts
+			(xy 43.18 54.61) (xy 43.18 58.42)
+		)
+		(stroke
+			(width 0)
+			(type default)
+		)
+	)
+	(wire
+		(pts
 			(xy 195.58 77.47) (xy 195.58 87.63)
 		)
@@
 	(wire
 		(pts
-			(xy 59.69 71.12) (xy 90.17 71.12)
+			(xy 59.69 71.12) (xy 81.28 71.12)
 		)
 		(stroke
@@
 	(wire
 		(pts
+			(xy 43.18 58.42) (xy 64.77 58.42)
+		)
+		(stroke
+			(width 0)
+			(type default)
+		)
+	)
+	(wire
+		(pts
 			(xy 176.53 87.63) (xy 195.58 87.63)
 		)
@@
 	(wire
 		(pts
-			(xy 31.75 58.42) (xy 64.77 58.42)
+			(xy 31.75 58.42) (xy 43.18 58.42)
 		)
 		(stroke
@@
 	(wire
 		(pts
-			(xy 31.75 71.12) (xy 52.07 71.12)
+			(xy 31.75 71.12) (xy 40.64 71.12)
 		)
 		(stroke
@@
 	(global_label "R2P1"
 		(shape input)
-		(at 40.64 71.12 90)
+		(at 40.64 68.58 90)
 		(fields_autoplaced yes)
 		(effects
@@
 		)
 		(property "Intersheetrefs" "${INTERSHEET_REFS}"
-			(at 40.64 63.1758 90)
+			(at 40.64 60.6358 90)
 			(effects
 				(font
@@
 	(global_label "R3P1"
 		(shape input)
-		(at 40.64 58.42 90)
+		(at 43.18 54.61 90)
 		(fields_autoplaced yes)
 		(effects
@@
 		)
 		(property "Intersheetrefs" "${INTERSHEET_REFS}"
-			(at 40.64 50.4758 90)
+			(at 43.18 46.6658 90)
 			(effects
 				(font
@@
 	(global_label "R3P3"
 		(shape input)
-		(at 81.28 58.42 90)
+		(at 81.28 57.15 90)
 		(fields_autoplaced yes)
 		(effects
@@
 		)
 		(property "Intersheetrefs" "${INTERSHEET_REFS}"
-			(at 81.28 50.4758 90)
+			(at 81.28 49.2058 90)
 			(effects
 				(font
@@
 		)
 	)
-	(global_label "R2P2"
+	(global_label "R2P3"
 		(shape input)
-		(at 81.28 71.12 90)
+		(at 81.28 68.58 90)
 		(fields_autoplaced yes)
 		(effects
@@
 		)
 		(property "Intersheetrefs" "${INTERSHEET_REFS}"
-			(at 81.28 63.1758 90)
+			(at 81.28 60.6358 90)
 			(effects
 				(font
@@
 			)
 		)
-		(property "Footprint" "Package_TO_SOT_THT:TO-92_Inline"
+		(property "Footprint" "Package_TO_SOT_THT:TO-92L_Inline_Wide"
 			(at 143.51 43.815 0)
 			(effects
@@
 			)
 		)
-		(property "Footprint" "Package_TO_SOT_THT:TO-92L_Inline"
+		(property "Footprint" "Package_TO_SOT_THT:TO-92L_Inline_Wide"
 			(at 223.52 96.52 0)
 			(effects
@@
 			)
 		)
-		(property "Footprint" "Package_TO_SOT_THT:TO-92_Inline"
+		(property "Footprint" "Package_TO_SOT_THT:TO-92L_Inline_Wide"
 			(at 140.97 43.815 0)
 			(effects
